File: resources/KiCad/Skull-Project_1.0/PersonSensor.kicad_sch (KiCad schematic)
At the start: 5 parts

Commit message: move schematic pdf to root directory + minor change
Connections:
- new net: A1.~ (VIN), U3. (GND)
Changed lines of the file:
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@@
   (title_block
     (title "Skull-Project 1.0")
-    (date "2024-09-27")
+    (date "2024-09-28")
     (rev "1.0")
     (company "github.com/Mark-MDO47/Skull-Project")

Commit message: update to KiCad 8.0.7
Connections:
- new net: A1.~ (VIN), U3. (GND)

Commit message: KiCad V9.0.1
Connections:
- new net: A1.~ (D13), U3. (GND)

Commit message: latest KiCad
Connections:
- new net: A1.~ (D13), U3. (GND)
Changed lines of the file:
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@@
 	(title_block
 		(title "Skull-Project 1.0")
-		(date "2024-09-28")
+		(date "2025-05-04")
 		(rev "1.0")
 		(company "github.com/Mark-MDO47/Skull-Project")
